File: schematics/motor-control/motor-control.kicad_sch (KiCad schematic)
At the start: 5 parts, among them J1 Conn_01x02, U1 L293D, U2 ESP32-S3-DevKitC

Commit message: schematic update
Parts:
- removed J1: Conn_01x02, symbol Connector_Generic:Conn_01x02
- added D1: RED, symbol Device:LED
- added D2: GREEN, symbol Device:LED
- added D3: BLUE, symbol Device:LED
- added J2: Conn_01x02, symbol Connector_Generic:Conn_01x02
- added Q1: BPW40, LED_THT:LED_D5.0mm_Clear, symbol Sensor_Optical:BPW40
- added R1, R2: 100, symbol Device:R
- added R3: 240, symbol Device:R
- added R4: 10k, symbol Device:R
- added U3: L7805, symbol Regulator_Linear:L7805
Connections:
- net 5V_motor is gone; now on net 5V: U1.8 (VCC2)
- net 3V3: now also Q1.1 (C)
- net 5V: now also U3.3 (OUT)
- net GND: now also J2.2 (Pin_2), R1.2, R2.2, R3.2, R4.2, U3.2 (GND)
- net green_led: now reaches U2.12 (GPIO8/ADC1_CH7)
- net green_led: now also D2.2 (A)
- net red_led: now reaches U2.7 (GPIO7/ADC1_CH6)
- net red_led: now also D1.2 (A)
- net blue_led: now reaches U2.8 (GPIO15/ADC2_CH4/32K_P)
- net blue_led: now also D3.2 (A)
- net color_sensor: now reaches U2.9 (GPIO16/ADC2_CH5/32K_N)
- net color_sensor: now also Q1.2 (E), R4.1
- new net: D2.1 (K), R2.1
- new net: D3.1 (K), R3.1
- new net: D1.1 (K), R1.1
- new net: J2.1 (Pin_1), U3.1 (IN)
