File: schematics/schematic.kicad_sch (KiCad schematic)
At the start: 14 parts, among them J2 Conn_01x02, Q1 BPW40, U1 L293D, U2 ESP32-S3-DevKitC, U3 L7805

Commit message: schematic update: almost done
Parts:
- removed D1: RED, symbol Device:LED
- removed D2: GREEN, symbol Device:LED
- removed D3: BLUE, symbol Device:LED
- removed R1, R2: 100, symbol Device:R
- removed R3: 240, symbol Device:R
- removed R4: 10k, symbol Device:R
- added C1: 0.33 uF, symbol TR3_V1:C
- added C2: 0.1 uF, symbol TR3_V1:C
- added D1: IR204A, LED_THT:LED_D3.0mm_IRBlack, symbol LED:IR204A
- added ENABLE1: Enable Switch, TR3_V1:SW_DS04-254-2-01BK-SMT, symbol TR3_V1:SW_DIP_x01
- added J2, LED_BLU_1, LED_GRN_1, LED_RED_1: Conn_01x02, symbol Connector_Generic:Conn_01x02
- added PWR2: LED, TR3_V1:150080RS75000_WRE, symbol TR3_V1:LED
- added R10: 110 kΩ, symbol TR3_V1:R_US
- added R16: 1.5 kΩ, Resistor_SMD:R_0603_1608Metric_Pad0.98x0.95mm_HandSolder, symbol TR3_V1:R_US
- added R17: 4.7 MΩ, Resistor_SMD:R_0603_1608Metric_Pad0.98x0.95mm_HandSolder, symbol TR3_V1:R_US
- added R18: 2.56 MΩ, Resistor_SMD:R_0603_1608Metric_Pad0.98x0.95mm_HandSolder, symbol TR3_V1:R_US
- added R5, R6: 100 Ω, symbol TR3_V1:R_US
- added R7: 240 Ω, symbol TR3_V1:R_US
- added R8: 10 kΩ, symbol TR3_V1:R_US
- added R9: 110 Ω, symbol TR3_V1:R_US
- U2: footprint PCM_Espressif:ESP32-S3-DevKitC -> footprints_pretty:XCVR_ESP32-S3-DEVKITC-1-N8R2
- renumbered J_Motor_Left to J_Motor_Left1, J_Motor_Right to J_Motor_Right1, J2 to PWR1
Connections:
- net blue_led: now also R7.2
- net color_sensor: now also J2.2 (Pin_2), R8.2; no longer Q1.2 (E)
- net green_led: now also R6.2
- net red_led: now also R5.2
- net at U3.1 (IN): now also C1.2, ENABLE1.2; no longer PWR1.1 (Pin_1)
- net 3V3 renamed +3.3V
- net +3.3V: now also J2.1 (Pin_1), PWR2.2 (A)
- net 5V renamed +5V
- net +5V: now also C2.1
- net GND renamed Earth
- net Earth: now also C1.1, C2.2, D1.1 (K), LED_BLU_1.2 (Pin_2), LED_GRN_1.2 (Pin_2), LED_RED_1.2 (Pin_2), R10.1, R16.2, R18.1, R8.1
- new net: LED_GRN_1.1 (Pin_1), R6.1
- new net: D1.2 (A), R9.2
- new net: LED_RED_1.1 (Pin_1), R5.1
- new net: PWR2.1 (K), R16.1
- new net: LED_BLU_1.1 (Pin_1), R7.1
- new net battery_in: R17.1, R18.2
- new net battery_raw: ENABLE1.1, PWR1.1 (Pin_1), R17.2
- new net distance_sensor: Q1.2 (E), R10.2
- new net ir_led: R9.1
Other:
- note added: "Battery Management"
- note added: "Color Sensor"
- note added: "Distance Sensor"
- note added: "Motor Control"
- note added: "PWR INDICATOR"
- note added: "Power Management"
- note added: "connect phototransistor to this terminal"
- moved on the sheet: J_Motor_Left1, J_Motor_Right1, PWR1, U1, U2, U3

Commit message: schematic done
Parts:
- removed U2: ESP32-S3-DevKitC, footprints_pretty:XCVR_ESP32-S3-DEVKITC-1-N8R2, symbol PCM_Espressif:ESP32-S3-DevKitC
- added BATSTAT: LED, LED_SMD:LED_0201_0603Metric, symbol TR3_V1:LED
- added H1, H2: (no value), symbol schematic:22_pin_header
- added R19: 1.5 kΩ, Resistor_SMD:R_0201_0603Metric, symbol TR3_V1:R_US
- added U4: ESP32-S3-DEVKITC-1-N8R2, ESP32-S3-DEVKITC-1-N8R2:XCVR_ESP32-S3-DEVKITC-1-N8R2, symbol ESP32-S3-DEVKITC-1-N8R2:ESP32-S3-DEVKITC-1-N8R2
- C1, C2: footprint (none) -> Capacitor_SMD:C_0201_0603Metric
- PWR2: footprint TR3_V1:150080RS75000_WRE -> LED_SMD:LED_0201_0603Metric
- R10, R5, R6, R7, R8, R9: footprint (none) -> Resistor_SMD:R_0201_0603Metric
- R16: footprint Resistor_SMD:R_0603_1608Metric_Pad0.98x0.95mm_HandSolder -> Resistor_SMD:R_0201_0603Metric
Connections:
- net +3.3V: now also H1. (22), U4.J1_1 (3V3), U4.J1_2 (3V3)
- net +5V: now also U4.J1_21 (5V0)
- net Earth: now also BATSTAT.1 (K), H2. (22), U4.J1_22 (GND), U4.J3_1 (GND), U4.J3_21 (GND), U4.J3_22 (GND)
- net battery_in renamed J1_13
- net J1_13: now also H1. (22), U4.J1_13 (GPIO3)
- net blue_led renamed J1_8
- net J1_8: now also H1. (22), U4.J1_8 (GPIO15)
- net color_sensor renamed J1_6
- net J1_6: now also H1. (22), U4.J1_6 (GPIO6)
- net distance_sensor renamed J1_15
- net J1_15: now also H1. (22), U4.J1_15 (GPIO9)
- net green_led renamed J1_7
- net J1_7: now also H1. (22), U4.J1_7 (GPIO7)
- net ir_led renamed J1_12
- net J1_12: now also H1. (22), U4.J1_12 (GPIO8)
- net left_A renamed J3_6
- net J3_6: now also H2. (22), U4.J3_6 (MTMS/GPIO42)
- net left_B renamed J3_7
- net J3_7: now also H2. (22), U4.J3_7 (MTDI/GPIO41)
- net left_M1 renamed J3_19
- net J3_19: now also H2. (22), U4.J3_19 (USB_D+/GPIO20)
- net left_M2 renamed J1_4
- net J1_4: now also H1. (22), U4.J1_4 (GPIO4)
- net red_led renamed J1_9
- net J1_9: now also H1. (22), U4.J1_9 (GPIO16)
- net right_A renamed J3_5
- net J3_5: now also H2. (22), U4.J3_5 (GPIO2)
- net right_B renamed J3_4
- net J3_4: now also H2. (22), U4.J3_4 (GPIO1)
- net right_M1 renamed J3_9
- net J3_9: now also H2. (22), U4.J3_9 (MTCK/GPIO39)
- net right_M2 renamed J3_8
- net J3_8: now also H2. (22), U4.J3_8 (MTDO/GPIO40)
- new net: BATSTAT.2 (A), R19.2
- new net J1_10: H1. (22), U4.J1_10 (GPIO17)
- new net J1_11: H1. (22), U4.J1_11 (GPIO18)
- new net J1_14: H1. (22), U4.J1_14 (GPIO46)
- new net J1_16: H1. (22), U4.J1_16 (GPIO10)
- new net J1_17: H1. (22), R19.1, U4.J1_17 (GPIO11)
- new net J1_18: H1. (22), U4.J1_18 (GPIO12)
- new net J1_19: H1. (22), U4.J1_19 (GPIO13)
- new net J1_20: H1. (22), U4.J1_20 (GPIO14)
- new net J1_21: H1. (22)
- new net J1_22: H1. (22)
- new net J1_3: H1. (22), U4.J1_3 (RST)
- new net J1_5: H1. (22), U4.J1_5 (GPIO5)
- new net J3_1: H2. (22)
- new net J3_10: H2. (22), U4.J3_10 (GPIO38)
- new net J3_11: H2. (22), U4.J3_11 (GPIO37)
- new net J3_12: H2. (22), U4.J3_12 (GPIO36)
- new net J3_13: H2. (22), U4.J3_13 (GPIO35)
- new net J3_14: H2. (22), U4.J3_14 (GPIO0)
- new net J3_15: H2. (22), U4.J3_15 (GPIO45)
- new net J3_16: H2. (22), U4.J3_16 (GPIO48)
- new net J3_17: H2. (22), U4.J3_17 (GPIO47)
- new net J3_18: H2. (22), U4.J3_18 (GPIO21)
- new net J3_2: H2. (22), U4.J3_2 (U0TXD/GPIO43)
- new net J3_20: H2. (22), U4.J3_20 (USB_D-/GPIO19)
- new net J3_3: H2. (22), U4.J3_3 (U0RXD/GPIO44)
Other:
- note added: "MCU"
- note added: "Pin Connections"
- moved on the sheet: D1, J2, J_Motor_Left1, J_Motor_Right1, LED_BLU_1, LED_GRN_1, LED_RED_1, Q1, R10, R17, R18, R5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

Commit message: schematic updates
Parts:
- removed LED_BLU_1, LED_GRN_1, LED_RED_1: Conn_01x02, symbol Connector_Generic:Conn_01x02
- removed R5, R6: 100 Ω, Resistor_SMD:R_0201_0603Metric, symbol TR3_V1:R_US
- removed R7: 240 Ω, Resistor_SMD:R_0201_0603Metric, symbol TR3_V1:R_US
- removed R8: 10 kΩ, Resistor_SMD:R_0201_0603Metric, symbol TR3_V1:R_US
- added J1: Conn_01x04, symbol Connector_Generic:Conn_01x04
- BATSTAT1: renamed from BATSTAT; footprint LED_SMD:LED_0201_0603Metric -> LED_THT:LED_D5.0mm
- H1, H2: footprint (none) -> Connector_PinHeader_2.54mm:PinHeader_1x22_P2.54mm_Vertical
- PWR1: renamed from PWR2; footprint LED_SMD:LED_0201_0603Metric -> LED_THT:LED_D5.0mm
- Q1: footprint LED_THT:LED_D5.0mm_Clear -> LED_THT:LED_D5.0mm
- U4: footprint ESP32-S3-DEVKITC-1-N8R2:XCVR_ESP32-S3-DEVKITC-1-N8R2 -> footprints_pretty:XCVR_ESP32-S3-DEVKITC-1-N8R2
- renumbered PWR1 to BAT1
Connections:
- net +3.3V: now also H1.1, H1.2; no longer H1. (22)
- net +5V: now also H1.21
- net Earth: now also H1.22, H2.1, H2.21, H2.22, J1.4 (Pin_4); no longer H2. (22)
- net J1_10: now also H1.10; no longer H1. (22)
- net J1_11: now also H1.11; no longer H1. (22)
- net J1_12: now also H1.12; no longer H1. (22)
- net J1_13: now also H1.13; no longer H1. (22)
- net J1_14: now also H1.14; no longer H1. (22)
- net J1_15: now also H1.15; no longer H1. (22)
- net J1_16: now also H1.16; no longer H1. (22)
- net J1_17: now also H1.17; no longer H1. (22)
- net J1_18: now also H1.18; no longer H1. (22)
- net J1_19: now also H1.19; no longer H1. (22)
- net J1_20: now also H1.20; no longer H1. (22)
- net J1_3: now also H1.3; no longer H1. (22)
- net J1_4: now also H1.4; no longer H1. (22)
- net J1_5: now also H1.5; no longer H1. (22)
- net J1_6: now also H1.6; no longer H1. (22)
- net J1_7: now also H1.7, J1.2 (Pin_2); no longer H1. (22)
- net J1_8: now also H1.8, J1.3 (Pin_3); no longer H1. (22)
- net J1_9: now also H1.9, J1.1 (Pin_1); no longer H1. (22)
- net J3_10: now also H2.10; no longer H2. (22)
- net J3_11: now also H2.11; no longer H2. (22)
- net J3_12: now also H2.12; no longer H2. (22)
- net J3_13: now also H2.13; no longer H2. (22)
- net J3_14: now also H2.14; no longer H2. (22)
- net J3_15: now also H2.15; no longer H2. (22)
- net J3_16: now also H2.16; no longer H2. (22)
- net J3_17: now also H2.17; no longer H2. (22)
- net J3_18: now also H2.18; no longer H2. (22)
- net J3_19: now also H2.19; no longer H2. (22)
- net J3_2: now also H2.2; no longer H2. (22)
- net J3_20: now also H2.20; no longer H2. (22)
- net J3_3: now also H2.3; no longer H2. (22)
- net J3_4: now also H2.4; no longer H2. (22)
- net J3_5: now also H2.5; no longer H2. (22)
- net J3_6: now also H2.6; no longer H2. (22)
- net J3_7: now also H2.7; no longer H2. (22)
- net J3_8: now also H2.8; no longer H2. (22)
- net J3_9: now also H2.9; no longer H2. (22)
- removed net J1_21: H1. (22)
- removed net J1_22: H1. (22)
- removed net J3_1: H2. (22)
Other:
- moved on the sheet: BATSTAT1, D1, J2, J_Motor_Left1, J_Motor_Right1, Q1, R10, R17, R18, R19, R9, U1

Commit message: pcb basically done
Parts:
- removed J1: Conn_01x04, symbol Connector_Generic:Conn_01x04
- removed J_Motor_Left1, J_Motor_Right1: Pololu, symbol Connector_Generic:Conn_01x06
- added H3, H4, H5, H6: MountingHole, MountingHole:MountingHole_2.7mm_M2.5, symbol Mechanical:MountingHole
- added J10, J3, J4, J5, J6, J7, J8, J9: Conn_01x02, footprints_pretty:CONN2_282836-2_TEC, symbol Connector_Generic:Conn_01x02
- BAT1, J2: footprint (none) -> footprints_pretty:CONN2_282836-2_TEC
- ENABLE1: footprint TR3_V1:SW_DS04-254-2-01BK-SMT -> footprints_pretty:Single Position DIP Switch
- R17, R18: footprint Resistor_SMD:R_0603_1608Metric_Pad0.98x0.95mm_HandSolder -> Resistor_THT:R_Box_L14.0mm_W5.0mm_P9.00mm
- U3: footprint (none) -> Package_TO_SOT_THT:TO-220-3_Vertical
- renumbered D1 to IR_LED1, Q1 to IR_SENS1
Connections:
- net +3.3V: now also J6.1 (Pin_1), J9.1 (Pin_1)
- net Earth: now also J10.2 (Pin_2), J4.2 (Pin_2), J7.2 (Pin_2)
- net J1_7: now also J3.2 (Pin_2)
- net J1_8: now also J4.1 (Pin_1)
- net J1_9: now also J3.1 (Pin_1)
- net J3_4: now also J10.1 (Pin_1)
- net J3_5: now also J9.2 (Pin_2)
- net J3_6: now also J6.2 (Pin_2)
- net J3_7: now also J7.1 (Pin_1)
- net at U1.11 (3Y): now also J8.1 (Pin_1)
- net at U1.14 (4Y): now also J8.2 (Pin_2)
- net at U1.3 (1Y): now also J5.1 (Pin_1)
- net at U1.6 (2Y): now also J5.2 (Pin_2)
Other:
- note added: "Mounting Holes"

Commit message: all done
Parts:
- added CSR1, J11: Conn_01x02, footprints_pretty:CONN2_282836-2_TEC, symbol Connector_Generic:Conn_01x02
- added J1: Conn_01x04, Connector_PinHeader_2.54mm:PinHeader_1x04_P2.54mm_Vertical, symbol Connector_Generic:Conn_01x04
- renumbered J2 to CSL1
Connections:
- net +3.3V: now also CSR1.1 (Pin_1), J11.1 (Pin_1)
- net +5V: now also J1.1 (Pin_1), J1.2 (Pin_2), J1.3 (Pin_3), J1.4 (Pin_4), J11.2 (Pin_2)
- net J1_16: now also CSR1.2 (Pin_2)
Other:
- note added: "0"
- note added: "1"
- note added: "10"
- note added: "11"
- note added: "12"
- note added: "13"
- note added: "14"
- note added: "15"
- note added: "16"
- note added: "17"
- note added: "18"
- note added: "19"
- note added: "2"
- note added: "20"
- note added: "21"
- note added: "3"
- note added: "35"
- note added: "36"
- note added: "37"
- note added: "38"
- note added: "39"
- note added: "3V3"
- note added: "4"
- note added: "40"
- note added: "41"
- note added: "42"
- note added: "45"
- note added: "46"
- note added: "47"
- note added: "48"
- note added: "5"
- note added: "5V"
- note added: "6"
- note added: "7"
- note added: "8"
- note added: "9"
- note added: "GND"
- note added: "RST"
- note added: "RX"
- note added: "TX"
- note added: "connect phototransistor to these terminals"
- note removed: "connect phototransistor to this terminal"
- moved on the sheet: H3, H4, H5, H6, IR_LED1, IR_SENS1, R10, R9
